File: hardware/kicad/03_Buttons.kicad_sch (KiCad schematic)
At the start: 30 parts, among them J2 COIL_L, J3 COIL_M, J4 COIL_R, U4 DRV8231ADSGR, U5 DRV8231ADSGR, U6 DRV8231ADSGR

Commit message: Resolve KiCad component sourcing and missing footprints
Parts:
- J2, J3, J4: footprint (none) -> Connector_JST:JST_PH_B2B-PH-SM4-TB_1x02-1MP_P2.00mm_Vertical; Checked (none) -> 2026-09-08; JLCPCB Library Type (none) -> Extended; JLCPCB Part # (none) -> C265003; LCSC (none) -> C265003; MPN (none) -> B2B-PH-SM4-TBT(LF)(SN); Manufacturer (none) -> JST; Sourcing Status TBD - select 2-pin coil connector after mechanism/current v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 -> JLCPCB catalog verified; stock/quote refresh required; Supplier URL (none) -> https://jlcpcb.com/partdetail/JST-B2B_PH_SM4_TBT_LF_SN/C265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
Other:
- note added: "DRAFT 0.2 - CIRCUIT DEVELOPMENT ONLY - NOT FOR FABRICATION"
- note removed: "DRAFT 0.1 - CIRCUIT DEVELOPMENT ONLY - NOT FOR FABRICATION"
Changed lines of the file:
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@@
     (title "MagMouse - 03_Buttons")
     (date "2026-09-08")
-    (rev "0.1 DRAFT")
+    (rev "0.2 DRAFT")
     (company "MagMouse")
     (comment 1 "NOT FOR FABRICATION - unresolved circuits listed in README.md"))
@@
       (justify left top))
 )
-  (text "DRAFT 0.1 - CIRCUIT DEVELOPMENT ONLY - NOT FOR FABRICATION"
+  (text "DRAFT 0.2 - CIRCUIT DEVELOPMENT ONLY - NOT FOR FABRICATION"
     (at 20 24 0)
     (effects
@@
           (size 1.0 1.0))
         (justify left)))
-    (property "Footprint" ""
+    (property "Footprint" "Connector_JST:JST_PH_B2B-PH-SM4-TB_1x02-1MP_P2.00mm_Vertical"
       (at 368.3 53.34 0)
       (hide yes)
@@
           (size 1.0 1.0))
         (justify left)))
-    (property "Datasheet" ""
+    (property "Datasheet" "https://datasheet.lcsc.com/datasheet/pdf/91225f8a61c6f7b7821281d8757bf5b1.pdf?productCode=C2941743"
       (at 368.3 53.34 0)
       (hide yes)
@@
           (size 1.0 1.0))
         (justify left)))
-    (property "Manufacturer" ""
+    (property "Manufacturer" "JST"
       (at 368.3 53.34 0)
       (hide yes)
@@
           (size 1.0 1.0))
         (justify left)))
-    (property "MPN" ""
+    (property "MPN" "B2B-PH-SM4-TBT(LF)(SN)"
       (at 368.3 53.34 0)
       (hide yes)
@@
           (size 1.0 1.0))
         (justify left)))
-    (property "LCSC" ""
+    (property "LCSC" "C265003"
       (at 368.3 53.34 0)
       (hide yes)
@@
           (size 1.0 1.0))
         (justify left)))
-    (property "JLCPCB Part #" ""
+    (property "JLCPCB Part #" "C265003"
       (at 368.3 53.34 0)
       (hide yes)
@@
           (size 1.0 1.0))
         (justify left)))
-    (property "Sourcing Status" "TBD - select 2-pin coil connector after mechanism/current validation"
+    (property "Sourcing Status" "JLCPCB catalog verified; stock/quote refresh required"
       (at 368.3 53.34 0)
       (hide yes)
@@
           (size 1.0 1.0))
         (justify left)))
-    (property "Checked" ""
+    (property "Checked" "2026-09-08"
       (at 368.3 53.34 0)
       (hide yes)
@@
         (path "/5d73110b-42e6-5c5c-9841-c82d60f67640/584f5e2a-40d4-5188-83de-a1357f3244b0"
           (reference "J2")
-          (unit 1)))))
+          (unit 1))))
+    (property "Supplier URL" "https://jlcpcb.com/partdetail/JST-B2B_PH_SM4_TBT_LF_SN/C265003"
+      (at 368.3 53.34 0)
+      (hide yes)
+      (effects
+        (font
+          (size 1 1))
+        (justify left)))
+    (property "JLCPCB Library Type" "Extended"
+      (at 368.3 53.34 0)
+      (hide yes)
+      (effects
+        (font
+          (size 1 1))
+        (justify left))))
   (wire
     (pts
@@
           (size 1.0 1.0))
         (justify left)))
-    (property "Footprint" ""
+    (property "Footprint" "Connector_JST:JST_PH_B2B-PH-SM4-TB_1x02-1MP_P2.00mm_Vertical"
       (at 368.3 124.46000000000001 0)
       (hide yes)
@@
           (size 1.0 1.0))
         (justify left)))
-    (property "Datasheet" ""
+    (property "Datasheet" "https://datasheet.lcsc.com/datasheet/pdf/91225f8a61c6f7b7821281d8757bf5b1.pdf?productCode=C2941743"
       (at 368.3 124.46000000000001 0)
       (hide yes)
@@
           (size 1.0 1.0))
         (justify left)))
-    (property "Manufacturer" ""
+    (property "Manufacturer" "JST"
       (at 368.3 124.46000000000001 0)
       (hide yes)
@@
           (size 1.0 1.0))
         (justify left)))
-    (property "MPN" ""
+    (property "MPN" "B2B-PH-SM4-TBT(LF)(SN)"
       (at 368.3 124.46000000000001 0)
       (hide yes)
@@
           (size 1.0 1.0))
         (justify left)))
-    (property "LCSC" ""
+    (property "LCSC" "C265003"
       (at 368.3 124.46000000000001 0)
       (hide yes)
@@
           (size 1.0 1.0))
         (justify left)))
-    (property "JLCPCB Part #" ""
+    (property "JLCPCB Part #" "C265003"
       (at 368.3 124.46000000000001 0)
       (hide yes)
@@
           (size 1.0 1.0))
         (justify left)))
-    (property "Sourcing Status" "TBD - select 2-pin coil connector after mechanism/current validation"
+    (property "Sourcing Status" "JLCPCB catalog verified; stock/quote refresh required"
       (at 368.3 124.46000000000001 0)
       (hide yes)
@@
           (size 1.0 1.0))
         (justify left)))
-    (property "Checked" ""
+    (property "Checked" "2026-09-08"
       (at 368.3 124.46000000000001 0)
       (hide yes)
@@
         (path "/5d73110b-42e6-5c5c-9841-c82d60f67640/584f5e2a-40d4-5188-83de-a1357f3244b0"
           (reference "J3")
-          (unit 1)))))
+          (unit 1))))
+    (property "Supplier URL" "https://jlcpcb.com/partdetail/JST-B2B_PH_SM4_TBT_LF_SN/C265003"
+      (at 368.3 124.46000000000001 0)
+      (hide yes)
+      (effects
+        (font
+          (size 1 1))
+        (justify left)))
+    (property "JLCPCB Library Type" "Extended"
+      (at 368.3 124.46000000000001 0)
+      (hide yes)
+      (effects
+        (font
+          (size 1 1))
+        (justify left))))
   (wire
     (pts
@@
           (size 1.0 1.0))
         (justify left)))
-    (property "Footprint" ""
+    (property "Footprint" "Connector_JST:JST_PH_B2B-PH-SM4-TB_1x02-1MP_P2.00mm_Vertical"
       (at 368.3 195.57999999999998 0)
       (hide yes)
@@
           (size 1.0 1.0))
         (justify left)))
-    (property "Datasheet" ""
+    (property "Datasheet" "https://datasheet.lcsc.com/datasheet/pdf/91225f8a61c6f7b7821281d8757bf5b1.pdf?productCode=C2941743"
       (at 368.3 195.57999999999998 0)
       (hide yes)
@@
           (size 1.0 1.0))
         (justify left)))
-    (property "Manufacturer" ""
+    (property "Manufacturer" "JST"
       (at 368.3 195.57999999999998 0)
       (hide yes)
@@
           (size 1.0 1.0))
         (justify left)))
-    (property "MPN" ""
+    (property "MPN" "B2B-PH-SM4-TBT(LF)(SN)"
       (at 368.3 195.57999999999998 0)
       (hide yes)
@@
           (size 1.0 1.0))
         (justify left)))
-    (property "LCSC" ""
+    (property "LCSC" "C265003"
       (at 368.3 195.57999999999998 0)
       (hide yes)
@@
           (size 1.0 1.0))
         (justify left)))
-    (property "JLCPCB Part #" ""
+    (property "JLCPCB Part #" "C265003"
       (at 368.3 195.57999999999998 0)
       (hide yes)
@@
           (size 1.0 1.0))
         (justify left)))
-    (property "Sourcing Status" "TBD - select 2-pin coil connector after mechanism/current validation"
+    (property "Sourcing Status" "JLCPCB catalog verified; stock/quote refresh required"
       (at 368.3 195.57999999999998 0)
       (hide yes)
@@
           (size 1.0 1.0))
         (justify left)))
-    (property "Checked" ""
+    (property "Checked" "2026-09-08"
       (at 368.3 195.57999999999998 0)
       (hide yes)
@@
         (path "/5d73110b-42e6-5c5c-9841-c82d60f67640/584f5e2a-40d4-5188-83de-a1357f3244b0"
           (reference "J4")
-          (unit 1)))))
+          (unit 1))))
+    (property "Supplier URL" "https://jlcpcb.com/partdetail/JST-B2B_PH_SM4_TBT_LF_SN/C265003"
+      (at 368.3 195.57999999999998 0)
+      (hide yes)
+      (effects
+        (font
+          (size 1 1))
+        (justify left)))
+    (property "JLCPCB Library Type" "Extended"
+      (at 368.3 195.57999999999998 0)
+      (hide yes)
+      (effects
+        (font
+          (size 1 1))
+        (justify left))))
   (wire
     (pts

Commit message: Implement USB-C power control schematic and validation
Connections:
- net ACT_5V_PENDING renamed ACT_5V
Other:
- note added: "DRAFT 0.3 - CIRCUIT DEVELOPMENT ONLY - NOT FOR FABRICATION"
- note added: "VREF nominal 1.65 V; IPROPI 1500 uA/A and 3.3k give Itrip approx 0.333 A. Provisional limit only: characterize accuracy at 5 V and low pulse currents. No continuous hold drive. IN1/IN2 are hardware-gated by ACT_DRIVE_EN; switched ACT_5V has reverse blocking and a local clamp. Current feedback is sampled directly; review settling/blanking before adding any filter to IPROPI."
- note removed: "DRAFT 0.2 - CIRCUIT DEVELOPMENT ONLY - NOT FOR FABRICATION"
- note removed: "VREF nominal 1.65 V; IPROPI 1500 uA/A and 3.3k give Itrip approx 0.333 A. Provisional limit only: characterize accuracy at 5 V and low pulse currents. No continuous hold drive. IN1/IN2 pulldowns provide reset default; hardware timeout + switched ACT supply are still missing. Current feedback is sampled directly; review settling/blanking before adding any filter to IPROPI."
Changed lines of the file:
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@@
     (title "MagMouse - 03_Buttons")
     (date "2026-09-08")
-    (rev "0.2 DRAFT")
+    (rev "0.3 DRAFT")
     (company "MagMouse")
     (comment 1 "NOT FOR FABRICATION - unresolved circuits listed in README.md"))
@@
       (justify left top))
 )
-  (text "DRAFT 0.2 - CIRCUIT DEVELOPMENT ONLY - NOT FOR FABRICATION"
+  (text "DRAFT 0.3 - CIRCUIT DEVELOPMENT ONLY - NOT FOR FABRICATION"
     (at 20 24 0)
     (effects
@@
       (type default))
 )
-  (global_label "ACT_5V_PENDING"
+  (global_label "ACT_5V"
     (shape bidirectional)
     (at 119.38 43.18 90)
@@
       (type default))
 )
-  (global_label "ACT_5V_PENDING"
+  (global_label "ACT_5V"
     (shape bidirectional)
     (at 271.78 49.53 90)
@@
       (type default))
 )
-  (global_label "ACT_5V_PENDING"
+  (global_label "ACT_5V"
     (shape bidirectional)
     (at 312.42 49.53 90)
@@
       (type default))
 )
-  (global_label "ACT_5V_PENDING"
+  (global_label "ACT_5V"
     (shape bidirectional)
     (at 119.38 114.3 90)
@@
       (type default))
 )
-  (global_label "ACT_5V_PENDING"
+  (global_label "ACT_5V"
     (shape bidirectional)
     (at 271.78 120.65 90)
@@
       (type default))
 )
-  (global_label "ACT_5V_PENDING"
+  (global_label "ACT_5V"
     (shape bidirectional)
     (at 312.42 120.65 90)
@@
       (type default))
 )
-  (global_label "ACT_5V_PENDING"
+  (global_label "ACT_5V"
     (shape bidirectional)
     (at 119.38 185.42 90)
@@
       (type default))
 )
-  (global_label "ACT_5V_PENDING"
+  (global_label "ACT_5V"
     (shape bidirectional)
     (at 271.78 191.77 90)
@@
       (type default))
 )
-  (global_label "ACT_5V_PENDING"
+  (global_label "ACT_5V"
     (shape bidirectional)
     (at 312.42 191.77 90)
@@
       (justify right))
 )
-  (text "VREF nominal 1.65 V; IPROPI 1500 uA/A and 3.3k give Itrip approx 0.333 A.\nProvisional limit only: characterize accuracy at 5 V and low pulse currents. No continuous hold drive.\nIN1/IN2 pulldowns provide reset default; hardware timeout + switched ACT supply are still missing.\nCurrent feedback is sampled directly; review settling/blanking before adding any filter to IPROPI."
+  (text "VREF nominal 1.65 V; IPROPI 1500 uA/A and 3.3k give Itrip approx 0.333 A.\nProvisional limit only: characterize accuracy at 5 V and low pulse currents. No continuous hold drive.\nIN1/IN2 are hardware-gated by ACT_DRIVE_EN; switched ACT_5V has reverse blocking and a local clamp.\nCurrent feedback is sampled directly; review settling/blanking before adding any filter to IPROPI."
     (at 20 248 0)
     (effects

Commit message: Allocate ESP32-S3 GPIO and peripheral resources
Other:
- note added: "DRAFT 0.4 - CIRCUIT DEVELOPMENT ONLY - NOT FOR FABRICATION"
- note removed: "DRAFT 0.3 - CIRCUIT DEVELOPMENT ONLY - NOT FOR FABRICATION"
Changed lines of the file:
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@@
     (title "MagMouse - 03_Buttons")
     (date "2026-09-08")
-    (rev "0.3 DRAFT")
+    (rev "0.4 DRAFT")
     (company "MagMouse")
     (comment 1 "NOT FOR FABRICATION - unresolved circuits listed in README.md"))
@@
       (justify left top))
 )
-  (text "DRAFT 0.3 - CIRCUIT DEVELOPMENT ONLY - NOT FOR FABRICATION"
+  (text "DRAFT 0.4 - CIRCUIT DEVELOPMENT ONLY - NOT FOR FABRICATION"
     (at 20 24 0)
     (effects
