File: hardware/kicad/04_Sensing.kicad_sch (KiCad schematic)
At the start: 10 parts, among them U10 ADS7038IRTER, U7 TMAG5253BA2IQDMRR, U8 TMAG5253BA2IQDMRR, U9 TMAG5253BA2IQDMRR

Commit message: Resolve KiCad component sourcing and missing footprints
Parts:
- C19, C20, C21: value 1uF/16V -> 1uF/50V; Checked (none) -> 2026-09-08; JLCPCB Library Type (none) -> Basic; JLCPCB Part # (none) -> C15849; LCSC (none) -> C15849; MPN (none) -> CL10A105KB8NNNC; Manufacturer (none) -> Samsung Electro-Mechanics; Sourcing Status TBD - not orderable -> JLCPCB catalog verified; stock/quote refresh required; Supplier URL (none) -> https://jlcpcb.com/partdetail/16531-CL10A105KB8NNNC/C15849
- U10: Checked (none) -> 2026-09-08; JLCPCB Library Type (none) -> Extended; JLCPCB Part # (none) -> C2871580; LCSC (none) -> C2871580; Sourcing Status TBD - not orderable -> JLCPCB catalog verified; stock/quote refresh required; Supplier URL (none) -> https://jlcpcb.com/partdetail/C2871580
- U7, U8, U9: Checked (none) -> 2026-09-08; JLCPCB Library Type (none) -> Extended; JLCPCB Part # (none) -> C35414983; LCSC (none) -> C35414983; Sourcing Status TBD - not orderable -> JLCPCB catalog verified; stock/quote refresh required; Supplier URL (none) -> https://jlcpcb.com/partdetail/37141530-TMAG5253BA2IQDMRR/C3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
Other:
- note added: "AIN0-2: Hall position. AIN3-5: driver current feedback. AIN6/7 unused in this draft. Wheel phase-current acquisition remains open; do not assume two spare channels solve PWM sampling. Hall sensors share the ADC analog supply/reference. Verify magnet gaps and interference under drive. ADC/Hall JLC catalog IDs assigned. Final layout/stencil and magnetic placement need review."
- note added: "DRAFT 0.2 - CIRCUIT DEVELOPMENT ONLY - NOT FOR FABRICATION"
- note removed: "AIN0-2: Hall position. AIN3-5: driver current feedback. AIN6/7 unused in this draft. Wheel phase-current acquisition remains open; do not assume two spare channels solve PWM sampling. Hall sensors share the ADC analog supply/reference. Verify magnet gaps and interference under drive. ADC/Hall MPNs and pin maps are selected; JLC sourcing and footprint sign-off remain pending."
- note removed: "DRAFT 0.1 - CIRCUIT DEVELOPMENT ONLY - NOT FOR FABRICATION"

Commit message: Implement USB-C power control schematic and validation
Connections:
- net +3V3: no longer U7.3 (EN), U8.3 (EN), U9.3 (EN)
- net USB_IMON_ADC: now reaches U10.5 (AIN6)
- net ACT_VMON: now reaches U10.6 (AIN7)
- new net HALL_EN: U7.3 (EN), U8.3 (EN), U9.3 (EN)
- no-connect marks 2 -> 0
Other:
- note added: "AIN0-2: Hall position. AIN3-5: button current. AIN6: input current. AIN7: actuator rail voltage. Wheel phase-current acquisition needs a separate path; no ADC inputs remain free. Hall sensors share the ADC supply/reference. Validate acquisition settling and magnetic interference. Power telemetry calibration and fault-injection tests are specified in docs/power.md."
- note added: "DRAFT 0.3 - CIRCUIT DEVELOPMENT ONLY - NOT FOR FABRICATION"
- note removed: "AIN0-2: Hall position. AIN3-5: driver current feedback. AIN6/7 unused in this draft. Wheel phase-current acquisition remains open; do not assume two spare channels solve PWM sampling. Hall sensors share the ADC analog supply/reference. Verify magnet gaps and interference under drive. ADC/Hall JLC catalog IDs assigned. Final layout/stencil and magnetic placement need review."
- note removed: "DRAFT 0.2 - CIRCUIT DEVELOPMENT ONLY - NOT FOR FABRICATION"
Changed lines of the file:
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@@
     (title "MagMouse - 04_Sensing")
     (date "2026-09-08")
-    (rev "0.2 DRAFT")
+    (rev "0.3 DRAFT")
     (company "MagMouse")
     (comment 1 "NOT FOR FABRICATION - unresolved circuits listed in README.md"))
@@
       (justify left top))
 )
-  (text "DRAFT 0.2 - CIRCUIT DEVELOPMENT ONLY - NOT FOR FABRICATION"
+  (text "DRAFT 0.3 - CIRCUIT DEVELOPMENT ONLY - NOT FOR FABRICATION"
     (at 20 24 0)
     (effects
@@
       (type default))
 )
-  (global_label "+3V3"
+  (global_label "HALL_EN"
     (shape bidirectional)
     (at 38.1 60.96 180)
@@
       (type default))
 )
-  (global_label "+3V3"
+  (global_label "HALL_EN"
     (shape bidirectional)
     (at 147.32 60.96 180)
@@
       (type default))
 )
-  (global_label "+3V3"
+  (global_label "HALL_EN"
     (shape bidirectional)
     (at 256.54 60.96 180)
@@
       (justify right))
 )
-  (no_connect
-    (at 101.6 190.5)
-)
-  (no_connect
-    (at 101.6 193.04)
-)
   (wire
     (pts
@@
       (justify right))
 )
-  (text "AIN0-2: Hall position. AIN3-5: driver current feedback. AIN6/7 unused in this draft.\nWheel phase-current acquisition remains open; do not assume two spare channels solve PWM sampling.\nHall sensors share the ADC analog supply/reference. Verify magnet gaps and interference under drive.\nADC/Hall JLC catalog IDs assigned. Final layout/stencil and magnetic placement need review."
+  (text "AIN0-2: Hall position. AIN3-5: button current. AIN6: input current. AIN7: actuator rail voltage.\nWheel phase-current acquisition needs a separate path; no ADC inputs remain free.\nHall sensors share the ADC supply/reference. Validate acquisition settling and magnetic interference.\nPower telemetry calibration and fault-injection tests are specified in docs/power.md."
     (at 20 243 0)
     (effects
@@
       (justify left top))
 )
-  (embedded_fonts no))
+  (embedded_fonts no)
+  (wire
+    (pts
+      (xy 101.6 190.5)
+      (xy 96.52 190.5))
+    (stroke
+      (width 0)
+      (type default))
+)
+  (global_label "USB_IMON_ADC"
+    (shape bidirectional)
+    (at 96.52 190.5 180)
+    (effects
+      (font
+        (size 1.0 1.0))
+      (justify right))
+)
+  (wire
+    (pts
+      (xy 101.6 193.04)
+      (xy 96.52 193.04))
+    (stroke
+      (width 0)
+      (type default))
+)
+  (global_label "ACT_VMON"
+    (shape bidirectional)
+    (at 96.52 193.04 180)
+    (effects
+      (font
+        (size 1.0 1.0))
+      (justify right))
+))

Commit message: Allocate ESP32-S3 GPIO and peripheral resources
Other:
- note added: "DRAFT 0.4 - CIRCUIT DEVELOPMENT ONLY - NOT FOR FABRICATION"
- note removed: "DRAFT 0.3 - CIRCUIT DEVELOPMENT ONLY - NOT FOR FABRICATION"
Changed lines of the file:
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@@
     (title "MagMouse - 04_Sensing")
     (date "2026-09-08")
-    (rev "0.3 DRAFT")
+    (rev "0.4 DRAFT")
     (company "MagMouse")
     (comment 1 "NOT FOR FABRICATION - unresolved circuits listed in README.md"))
@@
       (justify left top))
 )
-  (text "DRAFT 0.3 - CIRCUIT DEVELOPMENT ONLY - NOT FOR FABRICATION"
+  (text "DRAFT 0.4 - CIRCUIT DEVELOPMENT ONLY - NOT FOR FABRICATION"
     (at 20 24 0)
     (effects
