File: hardware/kicad/07_Power_Monitor.kicad_sch (KiCad schematic)
At the start: 25 parts, among them Q1 2N7002, Q2 2N7002, Q3 2N7002, U14 SN74LVC2G04DCKR, U19 TLV9001IDBVR

Commit message: Allocate ESP32-S3 GPIO and peripheral resources
Other:
- note added: "DRAFT 0.4 - CIRCUIT DEVELOPMENT ONLY - NOT FOR FABRICATION"
- note removed: "DRAFT 0.3 - CIRCUIT DEVELOPMENT ONLY - NOT FOR FABRICATION"
Changed lines of the file:
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@@
     (title "MagMouse - 07_Power_Monitor")
     (date "2026-09-08")
-    (rev "0.3 DRAFT")
+    (rev "0.4 DRAFT")
     (company "MagMouse")
     (comment 1 "NOT FOR FABRICATION - unresolved circuits listed in README.md"))
@@
       (justify left top))
 )
-  (text "DRAFT 0.3 - CIRCUIT DEVELOPMENT ONLY - NOT FOR FABRICATION"
+  (text "DRAFT 0.4 - CIRCUIT DEVELOPMENT ONLY - NOT FOR FABRICATION"
     (at 20 24 0)
     (effects
