File: hardware/kicad/02_MCU.kicad_sch (KiCad schematic)
At the start: 17 parts, among them SW1 RESET, SW2 BOOT, U3 ESP32-S3-MINI-1-N8

Commit message: Allocate ESP32-S3 GPIO and peripheral resources
Connections:
- net CS_IMU: now reaches U3.25 (IO21)
- net OPT_CTRL: now reaches U3.26 (IO26)
- net WHEEL_PWM_B: now reaches U3.27 (IO47)
- net MOTOR_SPI_MOSI: now reaches U3.28 (IO33)
- net MOTOR_SPI_SCLK: now reaches U3.29 (IO34)
- net WHEEL_PWM_C: now reaches U3.30 (IO48)
- net MOTOR_SPI_MISO: now reaches U3.31 (IO35)
- net CS_ADC2: now reaches U3.32 (IO36)
- net CS_MA735: now reaches U3.33 (IO37)
- net CS_DRV8316: now reaches U3.34 (IO38)
- net PAW_MOTION_N: now reaches U3.35 (IO39)
- net IMU_INT1: now reaches U3.36 (IO40)
- net DRV_FAULT_N: now reaches U3.37 (IO41)
- net WHEEL_PWM_A: now reaches U3.38 (IO42)
- net RGB_DATA: now reaches U3.41 (IO45)
- net BOOT_SAFE_SPARE: now reaches U3.44 (IO46)
- net CS_PAW: now reaches U3.6 (IO2)
- net WHEEL_RUN_REQ: now reaches U3.7 (IO3)
- no-connect marks 18 -> 0
Other:
- note added: "DRAFT 0.4 - CIRCUIT DEVELOPMENT ONLY - NOT FOR FABRICATION"
- note added: "GPIO allocation: 38 assigned + GPIO46 boot-low spare. Exact module: ESP32-S3-MINI-1-N8 (no PSRAM). SPI2: ADC1 / optical / IMU / angle / driver config. SPI3: dedicated ADC2. See sheet 09 and gpio-allocation.json. MCPWM0: wheel 3-PWM; MCPWM1: six independent button commands. RMT: one-wire RGB. GPIO3 wheel request and GPIO45 RGB have external pulldowns. GPIO26 is unavailable on N4R2. UART recovery r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"
- note removed: "DRAFT 0.3 - CIRCUIT DEVELOPMENT ONLY - NOT FOR FABRICATION"
- note removed: "GPIO4-9: button CMD signals through hardware AND gates. GPIO10-13: shared ADC SPI. GPIO1: VBUS_PRESENT_N; GPIO14/15: CC status; GPIO16/17: arm/heartbeat; GPIO18: sensors enable. USB remains GPIO19/20. Full wheel/optical/IMU/RGB pin and PWM budget still needs review."

Commit message: Add wheel control circuitry and autonomous regeneration brake
Parts:
- R5, R6: Checked 2026-09-08 -> 2026-09-09; JLCPCB Part # C23138 -> C23140; LCSC C23138 -> C23140; MPN 0603WAF3300T5E -> 0603WAF330JT5E; Sourcing Status LCSC listing verified; JLC stock check pending -> Corrected catalog mismatch: C23140 is 33 ohm; C23138 is 330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; Supplier URL https://www.lcsc.com/product-detail/C23138.html -> https://jlcpcb.com/partdetail/C23140
Changed lines of the file:
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@@
           (size 1.0 1.0))
         (justify left)))
-    (property "MPN" "0603WAF3300T5E"
+    (property "MPN" "0603WAF330JT5E"
       (at 218.44 165.1 0)
       (hide yes)
@@
           (size 1.0 1.0))
         (justify left)))
-    (property "LCSC" "C23138"
+    (property "LCSC" "C23140"
       (at 218.44 165.1 0)
       (hide yes)
@@
           (size 1.0 1.0))
         (justify left)))
-    (property "JLCPCB Part #" "C23138"
+    (property "JLCPCB Part #" "C23140"
       (at 218.44 165.1 0)
       (hide yes)
@@
           (size 1.0 1.0))
         (justify left)))
-    (property "Sourcing Status" "LCSC listing verified; JLC stock check pending"
+    (property "Sourcing Status" "Corrected catalog mismatch: C23140 is 33 ohm; C23138 is 330 ohm"
       (at 218.44 165.1 0)
       (hide yes)
@@
           (size 1.0 1.0))
         (justify left)))
-    (property "Checked" "2026-09-08"
+    (property "Checked" "2026-09-09"
       (at 218.44 165.1 0)
       (hide yes)
@@
           (size 1.0 1.0))
         (justify left)))
-    (property "Supplier URL" "https://www.lcsc.com/product-detail/C23138.html"
+    (property "Supplier URL" "https://jlcpcb.com/partdetail/C23140"
       (at 218.44 165.1 0)
       (hide yes)
@@
           (size 1.0 1.0))
         (justify left)))
-    (property "MPN" "0603WAF3300T5E"
+    (property "MPN" "0603WAF330JT5E"
       (at 289.56 165.1 0)
       (hide yes)
@@
           (size 1.0 1.0))
         (justify left)))
-    (property "LCSC" "C23138"
+    (property "LCSC" "C23140"
       (at 289.56 165.1 0)
       (hide yes)
@@
           (size 1.0 1.0))
         (justify left)))
-    (property "JLCPCB Part #" "C23138"
+    (property "JLCPCB Part #" "C23140"
       (at 289.56 165.1 0)
       (hide yes)
@@
           (size 1.0 1.0))
         (justify left)))
-    (property "Sourcing Status" "LCSC listing verified; JLC stock check pending"
+    (property "Sourcing Status" "Corrected catalog mismatch: C23140 is 33 ohm; C23138 is 330 ohm"
       (at 289.56 165.1 0)
       (hide yes)
@@
           (size 1.0 1.0))
         (justify left)))
-    (property "Checked" "2026-09-08"
+    (property "Checked" "2026-09-09"
       (at 289.56 165.1 0)
       (hide yes)
@@
           (size 1.0 1.0))
         (justify left)))
-    (property "Supplier URL" "https://www.lcsc.com/product-detail/C23138.html"
+    (property "Supplier URL" "https://jlcpcb.com/partdetail/C23140"
       (at 289.56 165.1 0)
       (hide yes)
