File: hardware/kicad/05_Protected_Power.kicad_sch (KiCad schematic)
At the start: 23 parts, among them U12 TPS259470LRPWR, U13 TPS259470LRPWR

Commit message: Allocate ESP32-S3 GPIO and peripheral resources
Other:
- note added: "DRAFT 0.4 - CIRCUIT DEVELOPMENT ONLY - NOT FOR FABRICATION"
- note removed: "DRAFT 0.3 - CIRCUIT DEVELOPMENT ONLY - NOT FOR FABRICATION"
Changed lines of the file:
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@@
     (title "MagMouse - 05_Protected_Power")
     (date "2026-09-08")
-    (rev "0.3 DRAFT")
+    (rev "0.4 DRAFT")
     (company "MagMouse")
     (comment 1 "NOT FOR FABRICATION - unresolved circuits listed in README.md"))
@@
       (justify left top))
 )
-  (text "DRAFT 0.3 - CIRCUIT DEVELOPMENT ONLY - NOT FOR FABRICATION"
+  (text "DRAFT 0.4 - CIRCUIT DEVELOPMENT ONLY - NOT FOR FABRICATION"
     (at 20 24 0)
     (effects

Commit message: Route input power and Type-C detection, select PCB stackup
Parts:
- added C88: 10uF/25V, Capacitor_SMD:C_0805_2012Metric, symbol Device:C
Connections:
- net GND: now also C88.2
- net PWR_5V: now also C88.1
Other:
- note added: "C88: local U12 output bypass. C1 remains beside the buck; do not rely on the long feed as local decoupling."
Changed lines of the file:
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@@
       (justify left top))
 )
-  (embedded_fonts no))
+  (embedded_fonts no)
+  (symbol
+    (lib_id "Device:C")
+    (at 86.36 165.1 0)
+    (unit 1)
+    (in_bom yes)
+    (on_board yes)
+    (dnp no)
+    (property "Reference" "C88"
+      (at 90.36 163.6 0)
+      (effects
+        (font
+          (size 1.0 1.0))
+        (justify left)))
+    (property "Value" "10uF/25V"
+      (at 90.36 166.1 0)
+      (effects
+        (font
+          (size 1.0 1.0))
+        (justify left)))
+    (property "Footprint" "Capacitor_SMD:C_0805_2012Metric"
+      (at 86.36 165.1 0)
+      (hide yes)
+      (effects
+        (font
+          (size 1.0 1.0))
+        (justify left)))
+    (property "Datasheet" ""
+      (at 86.36 165.1 0)
+      (hide yes)
+      (effects
+        (font
+          (size 1.0 1.0))
+        (justify left)))
+    (property "Manufacturer" "Samsung Electro-Mechanics"
+      (at 86.36 165.1 0)
+      (hide yes)
+      (effects
+        (font
+          (size 1.0 1.0))
+        (justify left)))
+    (property "MPN" "CL21A106KAYNNNE"
+      (at 86.36 165.1 0)
+      (hide yes)
+      (effects
+        (font
+          (size 1.0 1.0))
+        (justify left)))
+    (property "LCSC" "C15850"
+      (at 86.36 165.1 0)
+      (hide yes)
+      (effects
+        (font
+          (size 1.0 1.0))
+        (justify left)))
+    (property "JLCPCB Part #" "C15850"
+      (at 86.36 165.1 0)
+      (hide yes)
+      (effects
+        (font
+          (size 1.0 1.0))
+        (justify left)))
+    (property "Sourcing Status" "Reuses existing 10uF output capacitor selection; DC bias and order stock require review"
+      (at 86.36 165.1 0)
+      (hide yes)
+      (effects
+        (font
+          (size 1.0 1.0))
+        (justify left)))
+    (property "Checked" "2026-09-08"
+      (at 86.36 165.1 0)
+      (hide yes)
+      (effects
+        (font
+          (size 1.0 1.0))
+        (justify left)))
+    (property "Supplier URL" "https://www.lcsc.com/product-detail/C15850.html"
+      (at 86.36 165.1 0)
+      (hide yes)
+      (effects
+        (font
+          (size 1.0 1.0))
+        (justify left)))
+    (instances
+      (project "MagMouse"
+        (path "/5d73110b-42e6-5c5c-9841-c82d60f67640/8a66e1fe-51be-562e-9512-bb5cf22fe456"
+          (reference "C88")
+          (unit 1)))))
+  (wire
+    (pts
+      (xy 86.36 161.29)
+      (xy 86.36 156.21))
+    (stroke
+      (width 0)
+      (type default))
+)
+  (global_label "PWR_5V"
+    (shape bidirectional)
+    (at 86.36 156.21 90)
+    (effects
+      (font
+        (size 1.0 1.0))
+      (justify left))
+)
+  (wire
+    (pts
+      (xy 86.36 168.91)
+      (xy 86.36 173.99))
+    (stroke
+      (width 0)
+      (type default))
+)
+  (global_label "GND"
+    (shape bidirectional)
+    (at 86.36 173.99 270)
+    (effects
+      (font
+        (size 1.0 1.0))
+      (justify right))
+)
+  (text "C88: local U12 output bypass.\nC1 remains beside the buck; do not rely on the long feed as local decoupling."
+    (at 65 182 0)
+    (effects
+      (font
+        (size 1.0 1.0))
+      (justify left top))
+))

Commit message: Route U13 local actuator power and protection
Parts:
- added C89: 1uF/50V, Capacitor_SMD:C_0603_1608Metric, symbol Device:C
Connections:
- net GND: now also C89.2
- net PWR_5V: now also C89.1
Other:
- note added: "C89: local U13 input bypass. Place existing C40 at U13 OUT; C37-C39 remain rail storage."
Changed lines of the file:
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@@
+        (size 1.0 1.0))
+      (justify left top))
+)
+  (symbol
+    (lib_id "Device:C")
+    (at 312.42 165.1 0)
+    (unit 1)
+    (in_bom yes)
+    (on_board yes)
+    (dnp no)
+    (property "Reference" "C89"
+      (at 316.42 163.6 0)
+      (effects
+        (font
+          (size 1.0 1.0))
+        (justify left)))
+    (property "Value" "1uF/50V"
+      (at 316.42 166.1 0)
+      (effects
+        (font
+          (size 1.0 1.0))
+        (justify left)))
+    (property "Footprint" "Capacitor_SMD:C_0603_1608Metric"
+      (at 312.42 165.1 0)
+      (hide yes)
+      (effects
+        (font
+          (size 1.0 1.0))
+        (justify left)))
+    (property "Datasheet" ""
+      (at 312.42 165.1 0)
+      (hide yes)
+      (effects
+        (font
+          (size 1.0 1.0))
+        (justify left)))
+    (property "Manufacturer" "Samsung Electro-Mechanics"
+      (at 312.42 165.1 0)
+      (hide yes)
+      (effects
+        (font
+          (size 1.0 1.0))
+        (justify left)))
+    (property "MPN" "CL10A105KB8NNNC"
+      (at 312.42 165.1 0)
+      (hide yes)
+      (effects
+        (font
+          (size 1.0 1.0))
+        (justify left)))
+    (property "LCSC" "C15849"
+      (at 312.42 165.1 0)
+      (hide yes)
+      (effects
+        (font
+          (size 1.0 1.0))
+        (justify left)))
+    (property "JLCPCB Part #" "C15849"
+      (at 312.42 165.1 0)
+      (hide yes)
+      (effects
+        (font
+          (size 1.0 1.0))
+        (justify left)))
+    (property "Sourcing Status" "Reuses existing 1uF input capacitor selection; DC bias and order stock require review"
+      (at 312.42 165.1 0)
+      (hide yes)
+      (effects
+        (font
+          (size 1.0 1.0))
+        (justify left)))
+    (property "Checked" "2026-09-08"
+      (at 312.42 165.1 0)
+      (hide yes)
+      (effects
+        (font
+          (size 1.0 1.0))
+        (justify left)))
+    (property "Supplier URL" "https://www.lcsc.com/product-detail/C15849.html"
+      (at 312.42 165.1 0)
+      (hide yes)
+      (effects
+        (font
+          (size 1.0 1.0))
+        (justify left)))
+    (instances
+      (project "MagMouse"
+        (path "/5d73110b-42e6-5c5c-9841-c82d60f67640/8a66e1fe-51be-562e-9512-bb5cf22fe456"
+          (reference "C89")
+          (unit 1)))))
+  (wire
+    (pts
+      (xy 312.42 161.29)
+      (xy 312.42 156.21))
+    (stroke
+      (width 0)
+      (type default))
+)
+  (global_label "PWR_5V"
+    (shape bidirectional)
+    (at 312.42 156.21 90)
+    (effects
+      (font
+        (size 1.0 1.0))
+      (justify left))
+)
+  (wire
+    (pts
+      (xy 312.42 168.91)
+      (xy 312.42 173.99))
+    (stroke
+      (width 0)
+      (type default))
+)
+  (global_label "GND"
+    (shape bidirectional)
+    (at 312.42 173.99 270)
+    (effects
+      (font
+        (size 1.0 1.0))
+      (justify right))
+)
+  (text "C89: local U13 input bypass.\nPlace existing C40 at U13 OUT; C37-C39 remain rail storage."
+    (at 290 182 0)
+    (effects
+      (font
         (size 1.0 1.0))
       (justify left top))
