File: hardware/kicad/MagMouse.kicad_pcb (KiCad board)
At the start: 4 copper layers, 60 x 95 mm, 317 parts, among them J1 TYPE-C-31-M-12, J2 COIL_L, J3 COIL_M, J4 COIL_R, J5 GB1806 phase wires, J6 ENCODER_8P, Q1 2N7002, Q2 2N7002, Q3 2N7002, Q4 2N7002, Q5 AO3400A, SW1 RESET, SW2 BOOT, U1 TPD2EUSB30DRTR, U10 ADS7038IRTER, U11 TUSB320LAIRWBR, U12 TPS259470LRPWR, U13 TPS259470LRPWR, U14 SN74LVC2G04DCKR, U15 SN74LVC1G123DCUR, U16 SN74LVC08APWR, U17 SN74LVC08APWR, U18 SN74LVC08APWR, U19 TLV9001IDBVR, U2 TPS62162DSGR, U20 TPD2E2U06DCKR, U21 DRV8316RRGFR, U22 SN74LVC08APWR, U23 ADS7038IRTER, U24 SN74LVC125APWR, U25 SN74LVC125APWR, U26 SN74LVC125APWR, U28 TPS22919DCKR, U29 SN74LVC125APWR, U3 ESP32-S3-MINI-1-N8, U30 TLV1811DBVR, U31 LM4040AIM3-2.5/NOPB, U32 ICM-42688-P, U33 TPS7A2450DBVR, U34 SN74LV1T34DBVR, U35 PMW3360DM-T2QU, U36 TLV75519PDBVR, U37 SN74LVC125APWR, U38 TPS22918DBVR, U39 SN74LVC1G125DBVR, U4 DRV8231ADSGR, U5 DRV8231ADSGR, U6 DRV8231ADSGR, U7 TMAG5253BA2IQDMRR, U8 TMAG5253BA2IQDMRR, U9 TMAG5253BA2IQDMRR

Commit message: Route actuator power and analog sensing with layout checks
Parts:
- moved C59 2.55 mm to (138.2, 161.0), turned to 180 degrees
- moved C60 2.55 mm to (137.8, 163.5), turned to -90 degrees
- turned C61 to 180 degrees
Routing:
- net HALL_R: track 0.00 -> 121.9 mm, vias 0 -> 6
- net HALL_L: track 0.00 -> 58.7 mm, vias 0 -> 2
- net BTN_R_ISENSE: track 134.4 -> 81.7 mm, vias 7 -> 8
- net USB_IMON_BUF: track 108.7 -> 62.2 mm, vias 0 -> 3
- net HALL_M: track 0.00 -> 24.0 mm, vias 0 -> 2
- net USB_IMON_ADC: track 41.5 -> 18.1 mm, vias 4 -> 2
- net HALL_EN: track 219.3 -> 235.0 mm
- net BTN_M_VREF: track 27.1 -> 38.1 mm, vias 5 -> 7
- net GND: track 293.4 -> 299.3 mm
- net WHEEL_I_B: track 11.7 -> 7.45 mm, vias 2 -> 0
- net BTN_M_ISENSE: track 47.0 -> 50.5 mm, vias 3 -> 4
- net BTN_L_ISENSE: track 46.2 -> 49.4 mm
- net WHEEL_I_C: track 6.48 -> 5.34 mm, vias 2 -> 0
- net WHEEL_I_A: track 7.71 -> 7.82 mm, vias 2 -> 0
- added copper zone on B.Cu, net GND

Commit message: Review analog routing and plan modular assembly panel
Routing:
- net BTN_R_IN1: track 163.9 -> 71.0 mm, vias 9 -> 4
- net BTN_R_IN2: track 165.7 -> 75.0 mm, vias 10 -> 7
- net BTN_L_IN2: track 107.5 -> 59.8 mm, vias 4 -> 3
- net WHEEL_PWM_C: track 118.8 -> 97.3 mm
- net BRAKE_OUT: track 32.3 -> 12.3 mm
- net USB_IMON_BUF: track 62.2 -> 47.8 mm
- net BTN_R_ISENSE: track 81.7 -> 68.4 mm
- net WHEEL_PWM_A: track 69.3 -> 59.8 mm
- net BTN_M_VREF: track 38.1 -> 28.9 mm
- net WHEEL_PWM_B: track 93.8 -> 85.0 mm
- net BTN_M_ISENSE: track 50.5 -> 42.7 mm
- net DRV_INHA: track 42.5 -> 34.8 mm
- net BTN_L_ISENSE: track 49.4 -> 41.7 mm
- net DRV_INHB: track 59.0 -> 51.7 mm
- net ACT_VMON: track 23.7 -> 16.3 mm
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