File: hardware/modular/main/Main.kicad_pcb (KiCad board)
At the start: 4 copper layers, 80 x 125 mm, 246 parts, among them J1 TYPE-C-31-M-12, J10 WHEEL_POWER_2P, J2 COIL_L, J3 COIL_M, J4 COIL_R, J6 ENCODER_8P, J8 WHEEL_SIGNAL_30P, Q1 2N7002, Q2 2N7002, Q3 2N7002, SW1 RESET, SW2 BOOT, U1 TPD2EUSB30DRTR, U10 ADS7038IRTER, U11 TUSB320LAIRWBR, U12 TPS259470LRPWR, U13 TPS259470LRPWR, U14 SN74LVC2G04DCKR, U15 SN74LVC1G123DCUR, U16 SN74LVC08APWR, U17 SN74LVC08APWR, U18 SN74LVC08APWR, U19 TLV9001IDBVR, U2 TPS62162DSGR, U20 TPD2E2U06DCKR, U25 SN74LVC125APWR, U28 TPS22919DCKR, U29 SN74LVC125APWR, U3 ESP32-S3-MINI-1-N8, U32 ICM-42688-P, U33 TPS7A2450DBVR, U34 SN74LV1T34DBVR, U35 PMW3360DM-T2QU, U36 TLV75519PDBVR, U37 SN74LVC125APWR, U38 TPS22918DBVR, U39 SN74LVC1G125DBVR, U4 DRV8231ADSGR, U5 DRV8231ADSGR, U6 DRV8231ADSGR, U7 TMAG5253BA2IQDMRR, U8 TMAG5253BA2IQDMRR, U9 TMAG5253BA2IQDMRR

Commit message: Latest
Routing:
- net +3V3: track 0.00 -> 80.6 mm, vias 0 -> 4
- net VBUS_USB: track 0.00 -> 66.6 mm, vias 0 -> 8
- net PWR_5V: track 0.00 -> 55.0 mm, vias 0 -> 7
- net GND: track 0.00 -> 38.4 mm, vias 0 -> 32
- net USB_ILM: track 0.00 -> 22.9 mm, vias 0 -> 1
- net USB_UVLO: track 0.00 -> 10.2 mm
- net LOGIC_PG: track 0.00 -> 9.55 mm, vias 0 -> 2
- net USB_OVLO: track 0.00 -> 8.48 mm
- net ILM_HIGH_D: track 0.00 -> 6.02 mm
- net USB_FAULT_N: track 0.00 -> 5.48 mm
- net USB_DVDT: track 0.00 -> 5.08 mm
- net BUCK_SW: track 0.00 -> 3.95 mm
- net ILM_MED_D: track 0.00 -> 3.66 mm
- net USB_OV_2: track 0.00 -> 3.55 mm
- net USB_OV_1: track 0.00 -> 3.55 mm
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- added copper zone on F.Cu, net GND
- added copper zone on In1.Cu, net GND

Commit message: Complete shaped main PCB routing and return-path checks
Parts:
- moved TP1 59.5 mm to (70.9, 62.1)
- moved R68 48.1 mm to (57.0, 57.0), turned to 0 degrees
- moved C36 46.6 mm to (54.0, 49.0), turned to 0 degrees
- moved D4 43.5 mm to (53.0, 62.8)
- moved TP2 39.6 mm to (62.6, 80.6)
- moved TP24 38.7 mm to (32.5, 54.4)
- moved R67 38.5 mm to (48.0, 58.0)
- moved TP13 31.0 mm to (53.6, 93.8)
- moved TP6 24.9 mm to (62.0, 95.7)
- moved TP17 23.6 mm to (57.7, 78.8)
- moved TP23 16.8 mm to (34.7, 86.0)
- moved TP7 16.8 mm to (44.7, 100.8)
- moved R16 14.9 mm to (26.2, 53.0), turned to 0 degrees
- moved TP8 12.6 mm to (52.5, 96.0)
- moved TP4 12.1 mm to (30.8, 96.0)
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Routing:
- net +3V3: track 80.6 -> 582.0 mm, vias 4 -> 85
- net GND: track 38.4 -> 310.8 mm, vias 32 -> 254
- net ACT_5V: track 0.00 -> 244.2 mm, vias 0 -> 19
- net HALL_EN: track 0.00 -> 209.2 mm, vias 0 -> 17
- net MCU_EN: track 0.00 -> 176.7 mm, vias 0 -> 13
- net SPI_MOSI: track 0.00 -> 164.2 mm, vias 0 -> 15
- net USB_DP: track 0.00 -> 157.4 mm
- net USB_DM: track 0.00 -> 156.5 mm
- net RGB_DATA: track 0.00 -> 143.8 mm, vias 0 -> 3
- net CC_OUT1: track 0.00 -> 127.2 mm, vias 0 -> 9
- net OPT_3V3: track 0.00 -> 121.0 mm, vias 0 -> 11
- net CC_OUT2: track 0.00 -> 114.0 mm, vias 0 -> 10
- net VBUS_USB: track 66.6 -> 177.1 mm, vias 8 -> 16
- net PWR_5V: track 55.0 -> 160.2 mm, vias 7 -> 14
- net OPT_CTRL: track 0.00 -> 105.0 mm, vias 0 -> 16
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- added copper zone on B.Cu, net GND
- added copper zone on In2.Cu, net GND
Other:
- board text added: "MAIN 125 x 80 / 44 mm FRONT / ROUTED / MECHANICS PENDING"
- board text removed: "MAIN 125 x 80 / 44 mm FRONT / PLACEMENT DRAFT"
