File: hardware/modular/main/Main.kicad_pcb (KiCad board)
At the start: 4 copper layers, 80 x 125 mm, 246 parts, among them J1 TYPE-C-31-M-12, J10 WHEEL_POWER_2P, J2 COIL_L, J3 COIL_M, J4 COIL_R, J6 ENCODER_8P, J8 WHEEL_SIGNAL_30P, Q1 2N7002, Q2 2N7002, Q3 2N7002, SW1 RESET, SW2 BOOT, U1 TPD2EUSB30DRTR, U10 ADS7038IRTER, U11 TUSB320LAIRWBR, U12 TPS259470LRPWR, U13 TPS259470LRPWR, U14 SN74LVC2G04DCKR, U15 SN74LVC1G123DCUR, U16 SN74LVC08APWR, U17 SN74LVC08APWR, U18 SN74LVC08APWR, U19 TLV9001IDBVR, U2 TPS62162DSGR, U20 TPD2E2U06DCKR, U25 SN74LVC125APWR, U28 TPS22919DCKR, U29 SN74LVC125APWR, U3 ESP32-S3-MINI-1-N8, U32 ICM-42688-P, U33 TPS7A2450DBVR, U34 SN74LV1T34DBVR, U35 PMW3360DM-T2QU, U36 TLV75519PDBVR, U37 SN74LVC125APWR, U38 TPS22918DBVR, U39 SN74LVC1G125DBVR, U4 DRV8231ADSGR, U5 DRV8231ADSGR, U6 DRV8231ADSGR, U7 TMAG5253BA2IQDMRR, U8 TMAG5253BA2IQDMRR, U9 TMAG5253BA2IQDMRR

Commit message: Prepare wired Rev-A bench boards and submit manufacturing review
Parts:
- J10: value WHEEL_POWER_2P -> Soldered wires Power_1x02; footprint MagMouseModular:JST_PA_SM02B-PASS_1x02_P2.00mm_Horizontal -> MagMouseModular:Wire_Power_1x02_P2.54mm
- J2: value COIL_L -> Soldered wires Power_1x02; footprint Connector_JST:JST_PH_B2B-PH-SM4-TB_1x02-1MP_P2.00mm_Vertical -> MagMouseModular:Wire_Power_1x02_P2.54mm
- J3: value COIL_M -> Soldered wires Power_1x02; footprint Connector_JST:JST_PH_B2B-PH-SM4-TB_1x02-1MP_P2.00mm_Vertical -> MagMouseModular:Wire_Power_1x02_P2.54mm
- J4: value COIL_R -> Soldered wires Power_1x02; footprint Connector_JST:JST_PH_B2B-PH-SM4-TB_1x02-1MP_P2.00mm_Vertical -> MagMouseModular:Wire_Power_1x02_P2.54mm
- J6: value ENCODER_8P -> Soldered wires Signal_2x04; footprint Connector_JST:JST_SH_SM08B-SRSS-TB_1x08-1MP_P1.00mm_Horizontal -> MagMouseModular:Wire_Signal_2x04_P2.54mm
- J8: value WHEEL_SIGNAL_30P -> Soldered wires Signal_2x15; footprint Connector_FFC-FPC:Hirose_FH12-30S-0.5SH_1x30-1MP_P0.50mm_Horizontal -> MagMouseModular:Wire_Signal_2x15_P2.54mm
- L1: value SWPA4020S3R3MT -> SRP4020CC-3R3M; footprint Inductor_SMD:L_Sunlord_SWPA4020S -> MagMouseModular:L_Bourns_SRP4020CC
- moved TP10 54.4 mm to (53.0, 29.7)
- moved J10 49.0 mm to (71.0, 42.0), turned to 180 degrees
- moved J8 12.3 mm to (73.5, 63.5), turned to -90 degrees
- moved J6 2.50 mm to (28.0, 16.0)
- moved TP1 1.52 mm to (69.4, 62.1)
- moved J2 0.50 mm to (17.0, 35.5)
- moved J3 0.50 mm to (17.0, 60.5)
- moved J4 0.50 mm to (63.0, 35.5)
- moved L1 0.21 mm to (64.5, 23.4), turned to 90 degrees
- moved C2 0.15 mm to (67.8, 25.5)
Routing:
- net WHEEL_PWM_B: track 54.4 -> 137.0 mm, vias 8 -> 10
- net MOTOR_SPI_SCLK: track 67.3 -> 127.0 mm, vias 7 -> 11
- net WHEEL_PWM_A: track 52.9 -> 108.3 mm, vias 8 -> 11
- net CC_OUT1: track 127.2 -> 174.8 mm, vias 9 -> 11
- net ACT_5V: track 244.2 -> 200.7 mm, vias 19 -> 17
- net GND: track 310.8 -> 269.0 mm, vias 254 -> 259
- net WHEEL_RUN_REQ: track 53.2 -> 94.8 mm, vias 5 -> 9
- net RGB_DATA: track 143.8 -> 179.0 mm, vias 3 -> 5
- net SPI_SCLK: track 92.6 -> 126.1 mm, vias 9 -> 10
- net MOTOR_SPI_MOSI: track 52.1 -> 85.0 mm, vias 6 -> 11
- net VBUS_USB: track 177.1 -> 148.2 mm
- net CS_DRV8316: track 98.1 -> 126.6 mm, vias 12 -> 15
- net SPI_MOSI: track 164.2 -> 192.6 mm, vias 15 -> 16
- net DRV_FAULT_LOCAL_N: track 22.0 -> 46.4 mm, vias 5 -> 9
- net WHEEL_PWM_C: track 66.3 -> 43.7 mm, vias 7 -> 4
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