File: hardware/encoder/Encoder.kicad_sch (KiCad schematic)
At the start: 3 parts, among them J7 ENCODER_8P, U27 MA735GGU-P

Commit message: Prepare wired Rev-A bench boards and submit manufacturing review
Parts:
- J7: value ENCODER_8P -> Soldered wires Signal_2x04; footprint Connector_JST:JST_SH_SM08B-SRSS-TB_1x08-1MP_P1.00mm_Horizontal -> MagMouseModular:Wire_Signal_2x04_P2.54mm; JLCPCB Part # C160407 -> (none); LCSC C160407 -> (none); MPN SM08B-SRSS-TB(LF)(SN) -> (none); Manufacturer JST -> (none); Sourcing Status JLCPCB SMT listing checked 2026-09-09; order stock and harn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 -> Hand-soldered wire termination; no connector fitted; do not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; Supplier URL https://www.lcsc.com/product-detail/C160407.html -> (none)
Changed lines of the file:
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@@
           (size 1.0 1.0))
         (justify left)))
-    (property "Value" "ENCODER_8P"
+    (property "Value" "Soldered wires Signal_2x04"
       (at 70.04 79.74 0)
       (effects
@@
           (size 1.0 1.0))
         (justify left)))
-    (property "Footprint" "Connector_JST:JST_SH_SM08B-SRSS-TB_1x08-1MP_P1.00mm_Horizontal"
+    (property "Footprint" "MagMouseModular:Wire_Signal_2x04_P2.54mm"
       (at 66.04 78.74 0)
       (hide yes)
@@
           (size 1.0 1.0))
         (justify left)))
-    (property "Datasheet" "https://www.jst-mfg.com/product/pdf/eng/eSH.pdf"
+    (property "Datasheet" ""
       (at 66.04 78.74 0)
       (hide yes)
@@
           (size 1.0 1.0))
         (justify left)))
-    (property "Manufacturer" "JST"
+    (property "Manufacturer" ""
       (at 66.04 78.74 0)
       (hide yes)
@@
           (size 1.0 1.0))
         (justify left)))
-    (property "MPN" "SM08B-SRSS-TB(LF)(SN)"
+    (property "MPN" ""
       (at 66.04 78.74 0)
       (hide yes)
@@
           (size 1.0 1.0))
         (justify left)))
-    (property "LCSC" "C160407"
+    (property "LCSC" ""
       (at 66.04 78.74 0)
       (hide yes)
@@
           (size 1.0 1.0))
         (justify left)))
-    (property "JLCPCB Part #" "C160407"
+    (property "JLCPCB Part #" ""
       (at 66.04 78.74 0)
       (hide yes)
@@
           (size 1.0 1.0))
         (justify left)))
-    (property "Sourcing Status" "JLCPCB SMT listing checked 2026-09-09; order stock and harness fit need confirmation"
+    (property "Sourcing Status" "Hand-soldered wire termination; no connector fitted; do not fill these holes"
       (at 66.04 78.74 0)
       (hide yes)
@@
           (size 1.0 1.0))
         (justify left)))
-    (property "Supplier URL" "https://www.lcsc.com/product-detail/C160407.html"
+    (property "Supplier URL" ""
       (at 66.04 78.74 0)
       (hide yes)
