File: hardware/modular/wheel/18_Wheel_Harness.kicad_sch (KiCad schematic)
At the start: 8 parts, among them J11 WHEEL_POWER_2P, J9 WHEEL_SIGNAL_30P

Commit message: Prepare wired Rev-A bench boards and submit manufacturing review
Parts:
- J11: value WHEEL_POWER_2P -> Soldered wires Power_1x02; footprint MagMouseModular:JST_PA_SM02B-PASS_1x02_P2.00mm_Horizontal -> MagMouseModular:Wire_Power_1x02_P2.54mm; JLCPCB Part # C495198 -> (none); LCSC C495198 -> (none); MPN SM02B-PASS-TB(LF)(SN) -> (none); Manufacturer JST -> (none); Sourcing Status Catalog identity checked; stock and assembly quote not rese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 -> Hand-soldered wire termination; no connector fitted; do not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; Supplier URL https://jlcpcb.com/partdetail/C495198 -> (none)
- J9: value WHEEL_SIGNAL_30P -> Soldered wires Signal_2x15; footprint Connector_FFC-FPC:Hirose_FH12-30S-0.5SH_1x30-1MP_P0.50mm_Horizontal -> MagMouseModular:Wire_Signal_2x15_P2.54mm; JLCPCB Part # C506793 -> (none); LCSC C506793 -> (none); MPN FH12-30S-0.5SH(55) -> (none); Manufacturer Hirose -> (none); Sourcing Status Catalog identity checked; stock and assembly quote not rese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 -> Hand-soldered wire termination; no connector fitted; do not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; Supplier URL https://jlcpcb.com/partdetail/C506793 -> (none)
Changed lines of the file:
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@@
           (size 1 1))
         (justify left)))
-    (property "Value" "WHEEL_SIGNAL_30P"
+    (property "Value" "Soldered wires Signal_2x15"
       (at 96.44 101.1 0)
       (effects
@@
           (size 1 1))
         (justify left)))
-    (property "MPN" "FH12-30S-0.5SH(55)"
-      (at 96.44 101.6 0)
-      (hide yes)
-      (effects
-        (font
-          (size 1 1))
-        (justify left)))
-    (property "LCSC" "C506793"
-      (at 96.44 101.6 0)
-      (hide yes)
-      (effects
-        (font
-          (size 1 1))
-        (justify left)))
-    (property "JLCPCB Part #" "C506793"
-      (at 96.44 101.6 0)
-      (hide yes)
-      (effects
-        (font
-          (size 1 1))
-        (justify left)))
-    (property "Manufacturer" "Hirose"
-      (at 96.44 101.6 0)
-      (hide yes)
-      (effects
-        (font
-          (size 1 1))
-        (justify left)))
-    (property "Footprint" "Connector_FFC-FPC:Hirose_FH12-30S-0.5SH_1x30-1MP_P0.50mm_Horizontal"
-      (at 96.44 101.6 0)
-      (hide yes)
-      (effects
-        (font
-          (size 1 1))
-        (justify left)))
-    (property "Datasheet" "https://www.hirose.com/product/p/CL0586-0525-1-55"
+    (property "MPN" ""
+      (at 96.44 101.6 0)
+      (hide yes)
+      (effects
+        (font
+          (size 1 1))
+        (justify left)))
+    (property "LCSC" ""
+      (at 96.44 101.6 0)
+      (hide yes)
+      (effects
+        (font
+          (size 1 1))
+        (justify left)))
+    (property "JLCPCB Part #" ""
+      (at 96.44 101.6 0)
+      (hide yes)
+      (effects
+        (font
+          (size 1 1))
+        (justify left)))
+    (property "Manufacturer" ""
+      (at 96.44 101.6 0)
+      (hide yes)
+      (effects
+        (font
+          (size 1 1))
+        (justify left)))
+    (property "Footprint" "MagMouseModular:Wire_Signal_2x15_P2.54mm"
+      (at 96.44 101.6 0)
+      (hide yes)
+      (effects
+        (font
+          (size 1 1))
+        (justify left)))
+    (property "Datasheet" ""
       (at 96.44 101.6 0)
       (hide yes)
@@
           (size 1 1))
         (justify left)))
-    (property "Supplier URL" "https://jlcpcb.com/partdetail/C506793"
-      (at 96.44 101.6 0)
-      (hide yes)
-      (effects
-        (font
-          (size 1 1))
-        (justify left)))
-    (property "Sourcing Status" "Catalog identity checked; stock and assembly quote not reserved"
+    (property "Supplier URL" ""
+      (at 96.44 101.6 0)
+      (hide yes)
+      (effects
+        (font
+          (size 1 1))
+        (justify left)))
+    (property "Sourcing Status" "Hand-soldered wire termination; no connector fitted; do not fill these holes"
       (at 96.44 101.6 0)
       (hide yes)
@@
           (size 1 1))
         (justify left)))
-    (property "Value" "WHEEL_POWER_2P"
+    (property "Value" "Soldered wires Power_1x02"
       (at 203.12 55.38 0)
       (effects
@@
           (size 1 1))
         (justify left)))
-    (property "MPN" "SM02B-PASS-TB(LF)(SN)"
-      (at 203.12 55.88 0)
-      (hide yes)
-      (effects
-        (font
-          (size 1 1))
-        (justify left)))
-    (property "LCSC" "C495198"
-      (at 203.12 55.88 0)
-      (hide yes)
-      (effects
-        (font
-          (size 1 1))
-        (justify left)))
-    (property "JLCPCB Part #" "C495198"
-      (at 203.12 55.88 0)
-      (hide yes)
-      (effects
-        (font
-          (size 1 1))
-        (justify left)))
-    (property "Manufacturer" "JST"
-      (at 203.12 55.88 0)
-      (hide yes)
-      (effects
-        (font
-          (size 1 1))
-        (justify left)))
-    (property "Footprint" "MagMouseModular:JST_PA_SM02B-PASS_1x02_P2.00mm_Horizontal"
-      (at 203.12 55.88 0)
-      (hide yes)
-      (effects
-        (font
-          (size 1 1))
-        (justify left)))
-    (property "Datasheet" "https://www.jst-mfg.com/product/pdf/eng/ePA-F.pdf"
+    (property "MPN" ""
+      (at 203.12 55.88 0)
+      (hide yes)
+      (effects
+        (font
+          (size 1 1))
+        (justify left)))
+    (property "LCSC" ""
+      (at 203.12 55.88 0)
+      (hide yes)
+      (effects
+        (font
+          (size 1 1))
+        (justify left)))
+    (property "JLCPCB Part #" ""
+      (at 203.12 55.88 0)
+      (hide yes)
+      (effects
+        (font
+          (size 1 1))
+        (justify left)))
+    (property "Manufacturer" ""
+      (at 203.12 55.88 0)
+      (hide yes)
+      (effects
+        (font
+          (size 1 1))
+        (justify left)))
+    (property "Footprint" "MagMouseModular:Wire_Power_1x02_P2.54mm"
+      (at 203.12 55.88 0)
+      (hide yes)
+      (effects
+        (font
+          (size 1 1))
+        (justify left)))
+    (property "Datasheet" ""
       (at 203.12 55.88 0)
       (hide yes)
@@
           (size 1 1))
         (justify left)))
-    (property "Supplier URL" "https://jlcpcb.com/partdetail/C495198"
-      (at 203.12 55.88 0)
-      (hide yes)
-      (effects
-        (font
-          (size 1 1))
-        (justify left)))
-    (property "Sourcing Status" "Catalog identity checked; stock and assembly quote not reserved"
-      (at 203.12 55.88 0)
-      (hide yes)
+    (property "Supplier URL" ""
+      (at 203.12 55.88 0)
+      (hide yes)
+      (effects
+        (font
+          (size 1 1))
+        (justify left)))
+    (property "Sourcing Status" "Hand-soldered wire termination; no connector fitted; do not fill these holes"
+      (at 203.12 55.88 0)
+      (hide yes)
